File: pcb/kicad/openrz67.kicad_sch (KiCad schematic)
At the start: 61 parts, among them K1 G6K-2F-Y DC3, K2 G6K-2F-Y DC3, Q1 DTC114EKAT146, Q2 DTC114EKAT146, U1 ESP32-C3FH4, U3 LGS5500EP, U4 S4B-XH-A(LF)(SN), X1 40MHz, X2 32.768kHz

Commit message: KiCad: proper ERC pin types, mounting-hole symbols, courtyards, silk cleanup
- pin electrical types for ESP32-C3, LGS5500, ME6211 and USB-C; passives passive;
  PWR_FLAGs on GND/AGND/BAT+/VBUS/+5V_VIN/VDDA; ERC severities back to default
  (0 errors, 8 harmless dangling-wire warnings)
- symbol library pruned to the parts in use, embedded copies regenerated
- H1/H2: MountingHole symbols + MountingHole_2.0mm_Pad3.0 footprint, linked
- courtyards rebuilt from pads/body (+0.05 mm); 0402/0603 and overhanging
  connector silk moved to F.Fab; BOOT/EN label moved above the buttons
- tools/fetch_3d.sh bootstraps easyeda2kicad via uvx/pipx/venv; tools/export_step.sh
- DRC 0 errors / 0 unconnected / parity clean; 6 courtyard warnings remain
  where neighbours sit closer than 0.1 mm on the fabricated layout
Parts:
- added H1, H2: MountingHole, openrz67:MountingHole_2.0mm_Pad3.0, symbol openrz67:MountingHole

Commit message: Rev 2: battery connector on the bottom side, facing inward
BAT1 changes from the vertical THT B2B-PH-K-S to the SMD side-entry
S2B-PH-SM4-TB (LCSC C295747) on B.Cu at the left end, opening toward the
board centre, so the cell lies flat under the PCB and plugs in without a
lead bend. BAT+ is brought down with a 0.6/0.3 via next to C22; GND uses the
bottom pour. Five GND stitching vias under the new pads removed; bottom
silkscreen labels relocated. Symbol, footprint and 3D model added to the
project libraries. DRC 0 errors, parity clean; ERC unchanged.
Parts:
- BAT1: value B2B-PH-K-S(LF)(SN) -> S2B-PH-SM4-TB(LF)(SN); footprint openrz67:CONN-TH_B2B-PH-K-S -> openrz67:CONN-SMD_P2.00_S2B-PH-SM4-TB-LF-SN; symbol openrz67:B2B-PH-K-S(LF)(SN) -> openrz67:S2B-PH-SM4-TB; LCSC Part Name 1x2P 间距:2mm 直插 系列:PH -> 2P PH SMD side-entry 2.0mm; Manufacturer Part B2B-PH-K-S(LF)(SN) -> S2B-PH-SM4-TB(LF)(SN); Supplier Part C131337 -> C295747
Changed lines of the file:
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@@
+	(wire
+		(pts
+			(xy 118.11 69.85) (xy 118.11 72.39)
+		)
+		(stroke
+			(width 0)
+			(type default)
+		)
+	)
 	(wire
 		(pts
@@
 	)
 	(symbol
-		(lib_id "openrz67:B2B-PH-K-S(LF)(SN)")
-		(at 111.76 69.85 0)
+		(lib_id "openrz67:S2B-PH-SM4-TB")
+		(at 121.92 68.58 0)
 		(unit 1)
 		(body_style 0)
@@
 		(dnp no)
 		(property "Reference" "BAT1"
-			(at 105.41 64.77 0)
+			(at 115.57 63.50 0)
 			(show_name no)
 			(do_not_autoplace no)
@@
 			)
 		)
-		(property "Value" "B2B-PH-K-S(LF)(SN)"
-			(at 105.41 77.47 0)
+		(property "Value" "S2B-PH-SM4-TB(LF)(SN)"
+			(at 115.57 76.20 0)
 			(show_name no)
 			(do_not_autoplace no)
@@
 			)
 		)
-		(property "Footprint" "openrz67:CONN-TH_B2B-PH-K-S"
-			(at 111.76 69.85 0)
+		(property "Footprint" "openrz67:CONN-SMD_P2.00_S2B-PH-SM4-TB-LF-SN"
+			(at 121.92 68.58 0)
 			(hide yes)
 			(show_name no)
@@
 		)
 		(property "Datasheet" "https://atta.szlcsc.com/upload/public/pdf/source/20171026/C131342_15089839687311058815.pdf"
-			(at 111.76 69.85 0)
+			(at 121.92 68.58 0)
 			(hide yes)
 			(show_name no)
@@
 		)
 		(property "Description" ""
-			(at 111.76 69.85 0)
-			(hide yes)
-			(show_name no)
-			(do_not_autoplace no)
-			(effects
-				(font
-					(size 1.27 1.27)
-				)
-			)
-		)
-		(property "Manufacturer Part" "B2B-PH-K-S(LF)(SN)"
-			(at 111.76 69.85 0)
+			(at 121.92 68.58 0)
+			(hide yes)
+			(show_name no)
+			(do_not_autoplace no)
+			(effects
+				(font
+					(size 1.27 1.27)
+				)
+			)
+		)
+		(property "Manufacturer Part" "S2B-PH-SM4-TB(LF)(SN)"
+			(at 121.92 68.58 0)
 			(hide yes)
 			(show_name no)
@@
 		)
 		(property "Manufacturer" "JST"
-			(at 111.76 69.85 0)
-			(hide yes)
-			(show_name no)
-			(do_not_autoplace no)
-			(effects
-				(font
-					(size 1.27 1.27)
-				)
-			)
-		)
-		(property "Supplier Part" "C131337"
-			(at 111.76 69.85 0)
+			(at 121.92 68.58 0)
+			(hide yes)
+			(show_name no)
+			(do_not_autoplace no)
+			(effects
+				(font
+					(size 1.27 1.27)
+				)
+			)
+		)
+		(property "Supplier Part" "C295747"
+			(at 121.92 68.58 0)
 			(hide yes)
 			(show_name no)
@@
 		)
 		(property "Supplier" "LCSC"
-			(at 111.76 69.85 0)
-			(hide yes)
-			(show_name no)
-			(do_not_autoplace no)
-			(effects
-				(font
-					(size 1.27 1.27)
-				)
-			)
-		)
-		(property "LCSC Part Name" "1x2P 间距:2mm 直插 系列:PH"
-			(at 111.76 69.85 0)
-			(hide yes)
-			(show_name no)
+			(at 121.92 68.58 0)
+			(hide yes)
+			(show_name no)
+			(do_not_autoplace no)
+			(effects
+				(font
+					(size 1.27 1.27)
+				)
+			)
+		)
+		(property "LCSC Part Name" "2P PH SMD side-entry 2.0mm"
+			(at 121.92 68.58 0)
+			(hide yes)
+			(show_name no)

Commit message: Rev 2: widen board to 25 mm, add unpopulated 3-pin expansion header (GPIO4, 3V3, GND)
- new 3 mm strip along the back edge; outline rebuilt as a clean rounded rectangle
- J1 PinHeader 1x03 THT in the strip, excluded from BOM/POS; schematic Conn_01x03
  with global labels; GPIO4 = ESP32-C3 pad 9 (MTMS)
- GPIO4 routed F.Cu stub -> via -> B.Cu around the VCC track west end -> strip;
  3V3 stub to the bottom VCC track; a few GND/AGND stitching vias removed, two
  added to tie isolated top-pour islands down
- BAT1 nudged 0.15 mm off the front edge (0.3 mm copper-edge rule)
- S3 kept THT: neither SMD PH variant fits without moving C14/C28/D4
- DRC 0 errors / 0 unconnected / parity clean; ERC unchanged
Parts:
- added J1: EXP (not populated), openrz67:PinHeader_1x03_P2.54mm_Vertical, symbol openrz67:Conn_01x03
Connections:
- net GND: now also J1.3 (Pin_3)
- net VCC: now also J1.2 (Pin_2)
- net GPIO4: now reaches U1.9 (MTMS)
- net GPIO4: now also J1.1 (Pin_1)
Changed lines of the file:
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@@
+		)
+	)
+	(symbol
+		(lib_id "openrz67:Conn_01x03")
+		(at 398.78 80.01 0)
+		(unit 1)
+		(body_style 1)
+		(exclude_from_sim yes)
+		(in_bom no)
+		(on_board yes)
+		(in_pos_files no)
+		(dnp no)
+		(property "Reference" "J1"
+			(at 401.32 71.12 0)
+			(effects
+				(font
+					(size 1.27 1.27)
+				)
+			)
+		)
+		(property "Value" "EXP (not populated)"
+			(at 401.32 88.9 0)
+			(effects
+				(font
+					(size 1.27 1.27)
+				)
+			)
+		)
+		(property "Footprint" "openrz67:PinHeader_1x03_P2.54mm_Vertical"
+			(at 398.78 80.01 0)
+			(effects
+				(font
+					(size 1.27 1.27)
+				)
+				(hide yes)
+			)
+		)
+		(property "Datasheet" "~"
+			(at 398.78 80.01 0)
+			(effects
+				(font
+					(size 1.27 1.27)
+				)
+				(hide yes)
+			)
+		)
+		(property "Description" "Expansion header, not populated by default: GPIO4 3V3 GND"
+			(at 398.78 80.01 0)
+			(effects
+				(font
+					(size 1.27 1.27)
+				)
+				(hide yes)
+			)
+		)
+		(instances
+			(project "openrz67"
+				(path "/608428cc-ede5-4359-a9e7-0ca7713b40fb"
+					(reference "J1")
+					(unit 1)
+				)
+			)
+		)
+	)
+	(global_label "GPIO4"
+		(shape passive)
+		(at 393.7 77.47 180)
+		(effects
+			(font
+				(size 1.27 1.27)
+			)
+			(justify left)
+		)
+	)
+	(global_label "VCC"
+		(shape passive)
+		(at 393.7 80.01 180)
+		(effects
+			(font
+				(size 1.27 1.27)
+			)
+			(justify left)
+		)
+	)
+	(global_label "GND"
+		(shape passive)
+		(at 393.7 82.55 180)
+		(effects
+			(font
+				(size 1.27 1.27)
+			)
+			(justify left)
+		)
+	)
+	(global_label "GPIO4"
+		(shape passive)
+		(at 146.05 207.01 270)
+		(effects
+			(font
+				(size 1.27 1.27)
+			)
+			(justify left)
 		)
 	)

Commit message: J1: label GPIO4 / 3V3 / GND in silkscreen on both sides, header outline to F.Fab
Other:
- title: OpenRZ67 camera trigger -> openrz67-trigger

Commit message: Revert the 25 mm widening and the J1 expansion header
The header cost more than it bought. Reaching the new edge strip forced the
GPIO4 return path across the bottom pour, which split the B.Cu ground under
U1 and LDO1 off into a separate island and displaced three stitching vias
next to the antenna trace. One GPIO, on a header that was not going to be
populated, does not pay for that.

There is no cheap way back either: a through-hole pad needs both layers clear
at the same spot, and on this outline only two isolated positions qualify.
Bottom-side solder pads do fit, but the cell now occupies the bottom. It
belongs in the same pass as the enclosure rework, not before it.

- Board back to 48 x 22 mm; J1, its footprint and the GPIO4 net are gone from
  board, schematic and symbol library.
- B.Cu ground is one region of 649.5 mm2 holding both U1 and LDO1, and the
  antenna trace has 15 GND stitching vias again, the count it had before the
  header.
- Carried forward from 010d742 because they had nothing to do with the header:
  BAT1 sits 0.15 mm further off the board edge, and copper-to-edge 0.3 mm now
  actually reaches the zone filler. Without both, the reverted board fails DRC
  with an edge-clearance error on the BAT1 fixing pad.

Board and schematic hygiene in the same pass:

- Board title block added; the Gerber job file reported revision "rev?" and
  now reports 2.
- BAT+ / BAT- and the polarity mark raised to 1.067 mm, matching the board's
  other silkscreen. Every text now clears JLCPCB's 1.0 mm except the BOOT EN
  label, which cannot be enlarged where it sits; see README.
- BAT1 footprint silkscreen line 0.06 -> 0.15 mm, under the fab minimum.
- Two vias at 0.305 mm drill merged into the 0.300 mm tool: 7 drill tools -> 6.
- ERC is now 0 errors, 0 warnings. Removed an orphan S1/S2/AGND label cluster
  that connected nothing, and shortened three wire tails that ran past their
  labels. Netlist verified node-for-node before and after: 64 nets, identical.
- AGND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
Parts:
- removed J1: EXP (not populated), openrz67:PinHeader_1x03_P2.54mm_Vertical, symbol openrz67:Conn_01x03
Connections:
- net GPIO4: no longer names the net of U1.9 (MTMS)
Other:
- title: openrz67-trigger -> OpenRZ67 camera trigger

Commit message: Rev 2: decouple the ESP32-C3 analog supply behind the ferrite bead
L2 sits between VCC and U1 pins 31/32 (VDDA, radio and ADC supply), but every
3.3 V capacitor on the board was on the VCC side of it. A bead with no
capacitor behind it is just series impedance: the radio's transmit bursts have
to pull through it, and the noise it is meant to block has no path to ground.
Espressif's reference design puts 0.1 uF at those pins.

Rather than squeeze a new part into the 2 mm gap in front of the pins, reuse
C5, the 100 nF that already sat 1.2 mm from L2 pin 2: move it to the far side
of the bead. The net is now named VDDA.

- Schematic: C5 moved onto the L2 -> U1 wire, global label VDDA on that net.
- Board: C5 pad 1 on VDDA with a 0.16 mm track from L2 pad 2; the four VCC
  segments that fed L2 pin 1 through C5 are gone, replaced by a 0.45/0.25 via
  beside L2 pad 1 down to the existing B.Cu VCC track. B.Cu ground under U1
  stays one region (648.7 mm2).
- Same part, same position: BOM and position file are unchanged.

DRC 0 errors, the same 8 known warnings; schematic parity clean; ERC 0/0.
Connections:
- net VCC: no longer C5.1
- net VDDA: now reaches L2.2, U1.31 (VDDA), U1.32 (VDDA)
- net VDDA: now also C5.1
Other:
- moved on the sheet: C5
Changed lines of the file:
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@@
 	)
 	(junction
-		(at 119.38 140.97)
+		(at 142.24 140.97)
 		(diameter 0)
 		(color 0 0 0 0)
@@
 	)
 	(junction
-		(at 119.38 151.13)
+		(at 142.24 151.13)
 		(diameter 0)
 		(color 0 0 0 0)
@@
 	(wire
 		(pts
-			(xy 119.38 140.97) (xy 128.27 140.97)
+			(xy 105.41 140.97) (xy 128.27 140.97)
 		)
 		(stroke
@@
 	(wire
 		(pts
-			(xy 143.51 151.13) (xy 119.38 151.13)
+			(xy 143.51 151.13) (xy 105.41 151.13)
 		)
 		(stroke
@@
 	(wire
 		(pts
-			(xy 119.38 151.13) (xy 105.41 151.13)
-		)
-		(stroke
-			(width 0)
-			(type default)
-		)
-	)
-	(wire
-		(pts
 			(xy 163.83 149.86) (xy 176.53 149.86)
 		)
@@
 	(wire
 		(pts
-			(xy 119.38 140.97) (xy 105.41 140.97)
-		)
-		(stroke
-			(width 0)
-			(type default)
-		)
-	)
-	(wire
-		(pts
 			(xy 133.35 189.23) (xy 128.27 189.23)
 		)
@@
 		)
 	)
+	(global_label "VDDA"
+		(shape passive)
+		(at 139.7 140.97 0)
+		(effects
+			(font
+				(size 1.5748 1.5748)
+			)
+			(justify left bottom)
+		)
+	)
 	(global_label "+5V"
 		(shape passive)
@@
 	(symbol
 		(lib_id "openrz67:GRM155R71H104KE14D")
-		(at 119.38 146.05 270)
+		(at 142.24 146.05 270)
 		(unit 1)
 		(body_style 0)
@@
 		(dnp no)
 		(property "Reference" "C5"
-			(at 123.19 146.05 90)
+			(at 146.05 146.05 90)
 			(show_name no)
 			(do_not_autoplace no)
@@
 		)
 		(property "Value" "100nF"
-			(at 123.19 148.59 90)
+			(at 146.05 148.59 90)
 			(show_name no)
 			(do_not_autoplace no)
@@
 		)
 		(property "Footprint" "openrz67:C0402"
-			(at 119.38 146.05 0)
+			(at 142.24 146.05 0)
 			(hide yes)
 			(show_name no)
@@
 		)
 		(property "Datasheet" "https://atta.szlcsc.com/upload/public/pdf/source/20180326/C77020_39BD49C951FF1AF0DB1F1FAC5AC1E401.pdf"
-			(at 119.38 146.05 0)
+			(at 142.24 146.05 0)
 			(hide yes)
 			(show_name no)
@@
 		)
 		(property "Description" ""
-			(at 119.38 146.05 0)
+			(at 142.24 146.05 0)
 			(hide yes)
 			(show_name no)
@@
 		)
 		(property "Manufacturer Part" "GRM155R71H104KE14D"
-			(at 119.38 146.05 0)
+			(at 142.24 146.05 0)
 			(hide yes)
 			(show_name no)
@@
 		)
 		(property "Manufacturer" "muRata(村田)"
-			(at 119.38 146.05 0)
+			(at 142.24 146.05 0)
 			(hide yes)
 			(show_name no)
@@
 		)
 		(property "Supplier Part" "C77020"
-			(at 119.38 146.05 0)
+			(at 142.24 146.05 0)
 			(hide yes)
 			(show_name no)
@@
 		)
 		(property "Supplier" "LCSC"
-			(at 119.38 146.05 0)
+			(at 142.24 146.05 0)
 			(hide yes)
 			(show_name no)
@@
 		)
 		(property "LCSC Part Name" "100nF ±10% 50V"
-			(at 119.38 146.05 0)
+			(at 142.24 146.05 0)
 			(hide yes)
 			(show_name no)

Commit message: Rev 2: replace the G6K relays with TLP172GM PhotoMOS, fix the JLCPCB CPL format
Each shutter channel is now one Toshiba TLP172GM (LCSC C261926) with its LED
driven from the GPIO through 330 R (C25104). K1/K2, the DTC114E drivers, the
flyback diodes and the coil decoupling caps are gone: eight parts become four,
the tallest top-side part drops from 5.2 to 2.2 mm, and no coil current is
drawn while an exposure is held. Camera ground stays isolated: AGND touches
only U4 pin 2 and the two PhotoMOS outputs, and the AGND pours were pulled in
so the LED side sits in the GND domain.

R4/R5 (USB 22 R) move to UNI-ROYAL 0402WGF220JTCE (C25092, Basic); JLCPCB
had two of the Yageo part in stock.

regen.sh rewrites the position file into JLCPCB's CPL header layout; their
uploader rejects KiCad's native header.

DRC 0 errors / 7 known warnings, ERC 0/0, schematic parity clean.
Parts:
- removed C27, C28: 10uF, openrz67:C0603, symbol openrz67:CL10A106MA8NRNC
- removed D1, D2: 1N4148WT, openrz67:SOD-523_L1.2-W0.8-LS1.6-RD, symbol openrz67:1N4148WT_C232841
- removed K1, K2: G6K-2F-Y DC3, openrz67:RELAY-SMD_G6K-2F-Y, symbol openrz67:G6K-2F-Y3VDC
- removed Q1, Q2: DTC114EKAT146, openrz67:SOT-346_L2.9-W1.6-P1.90-LS2.8-TR-CW, symbol openrz67:DTC114EKAT146
- added R21, R22: 330Ω, openrz67:R0402, symbol openrz67:0402WGF3300TCE
- added U5, U6: TLP172GM, openrz67:SMD-4_L4.6-W3.7-P2.54-LS7.0-BR, symbol openrz67:TLP172GM
- R4, R5: symbol openrz67:RC0402JR-0722RL -> openrz67:0402WGF220JTCE; LCSC Part Name 厚膜电阻 22Ω ±5% 62.5mW -> 22Ω ±1% 62.5mW 厚膜电阻; Manufacturer YAGEO(国巨) -> UNI-ROYAL(厚声); Manufacturer Part RC0402JR-0722RL -> 0402WGF220JTCE; Supplier Part C93929 -> C25092
Connections:
- net AGND: now also U5.3 (D), U6.3 (D)
- net D1: now also R22.2
- net D6: now also R21.2
- net GND: now also U5.2 (K), U6.2 (K)
- net S1: now also U5.4 (D)
- net S2: now also U6.4 (D)
- new net: R21.1, U5.1 (A)
- new net: R22.1, U6.1 (A)
- no-connect marks 26 -> 18
Other:
- note added: "2x PhotoMOS"
- note removed: "2x Relays"

Commit message: Review follow-ups: S1 driver to GPIO4, 220 R LED resistors, S1_DRV/S2_DRV nets
GPIO21 is U0TXD and idles high from the ROM boot log until setup() runs, so
the S1 output was closed during every boot. Harmless on its own, since the
camera needs S1 and S2 together, but GPIO4 (U1 pin 9, free) is a plain input
at reset, and the move frees UART0 TX for logging. Firmware constants
renamed to shutterPinS1 = 4 / shutterPinS2 = 3; builds.

330 R gave 3.8 mA at worst-case VOH/VF, under Toshiba's 5 mA minimum; 220 R
(C25091, Basic) gives 5.6 mA worst case, 9 mA typical.

Nets D6/D1 (Wemos names) renamed S1_DRV/S2_DRV. The S2_DRV bottom-layer
diagonal moved 0.3 mm to make room for the new via next to U1 pin 10.

DRC 0 errors / 7 known warnings, ERC 0/0, parity clean.
Parts:
- R21, R22: value 330Ω -> 220Ω; symbol openrz67:0402WGF3300TCE -> openrz67:0402WGF2200TCE; LCSC Part Name 330Ω ±1% 62.5mW 厚膜电阻 -> 220Ω ±1% 62.5mW 厚膜电阻; Manufacturer Part 0402WGF3300TCE -> 0402WGF2200TCE; Supplier Part C25104 -> C25091
Connections:
- net S1_DRV: now reaches U1.9 (MTMS)
- net S1_DRV: now also R21.2
- net D1 renamed S2_DRV
- net D6: no longer names the net of U1.28 (U0TXD)
- net D6: no longer R21.2
Other:
- note added: "S1_DRV = GPIO4, S2_DRV = GPIO3 (src/main.cpp)"
- note removed: "const int shutterPin = D6; // Pin for trigger"
