File: nrf/kicad/openrz67-nrf.kicad_pcb (KiCad board)
At the start: 2 copper layers, 29.5 x 29 mm, 15 parts, among them J1 Camera, J2 SWD, Q1 AO3401A, SW1 B3U-1000P, U1 E73-2G4M08S1F, U2 TLP172AM, U3 TLP172AM

Commit message: nrf: camera connector in camera pin order (rev B)
Connections:
- J1 pad 1: CAM_GND -> unconnected-(J1-Pad1)
- J1 pad 2: unconnected-(J1-Pad2) -> CAM_GND
Routing:
- net CAM_GND: track 19.5 -> 20.0 mm
Other:
- board text added: "OpenRZ67 nRF rev B"
- board text removed: "OpenRZ67 nRF rev A"
